File: openDTU_wDisplay.kicad_pcb (KiCad board)
At the start: 2 copper layers, 104.1 x 50.3 mm, 9 parts

Commit message: Editorial changes
Change capacity to radial
Parts:
- C1: footprint Capacitor_THT:C_Axial_L3.8mm_D2.6mm_P7.50mm_Horizontal -> Capacitor_THT:C_Radial_D4.0mm_H5.0mm_P1.50mm
Other:
- board text added: "github.com/SteffMUC/openDTU_wDisplay [2023-01-27]"
- board text removed: "github.com/SteffMUC/openDTUwDisplay [2023-01-27]"
Changed lines of the file:
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@@
     )
   )
-  (footprint "Capacitor_THT:C_Axial_L3.8mm_D2.6mm_P7.50mm_Horizontal" (layer "F.Cu")
+  (footprint "Capacitor_THT:C_Radial_D4.0mm_H5.0mm_P1.50mm" (layer "F.Cu")
     (at 113.598 112.776)
-    (descr "C, Axial series, Axial, Horizontal, pin pitch=7.5mm, , length*diameter=3.8*2.6mm^2, http://www.vishay.com/docs/45231/arseries.pdf")
-    (tags "C Axial series Axial Horizontal pin pitch 7.5mm  length 3.8mm diameter 2.6mm")
+    (descr "C, Radial series, Radial, pin pitch=1.50mm, diameter=4mm, height=5mm, Non-Polar Electrolytic Capacitor")
+    (tags "C Radial series Radial pin pitch 1.50mm diameter 4mm height 5mm Non-Polar Electrolytic Capacitor")
     (property "Sheetfile" "openDTU_wDisplay.kicad_sch")
     (property "Sheetname" "")
     (attr through_hole)
-    (fp_text reference "C1" (at 7.306 2.54) (layer "F.SilkS")
-      (effects (font (size 1 1) (thickness 0.15)))
-    )
-    (fp_text value "10uF" (at 3.75 2.42) (layer "F.Fab")
-      (effects (font (size 1 1) (thickness 0.15)))
-    )
-    (fp_text user "${REFERENCE}" (at 3.75 0) (layer "F.Fab")
-      (effects (font (size 0.76 0.76) (thickness 0.114)))
-    )
-    (fp_line (start 1.04 0) (end 1.73 0) (layer "F.SilkS") (width 0.12))
-    (fp_line (start 5.77 1.42) (end 5.77 -1.42) (layer "F.SilkS") (width 0.12))
-    (fp_line (start 5.77 -1.42) (end 1.73 -1.42) (layer "F.SilkS") (width 0.12))
-    (fp_line (start 6.46 0) (end 5.77 0) (layer "F.SilkS") (width 0.12))
-    (fp_line (start 1.73 -1.42) (end 1.73 1.42) (layer "F.SilkS") (width 0.12))
-    (fp_line (start 1.73 1.42) (end 5.77 1.42) (layer "F.SilkS") (width 0.12))
-    (fp_line (start -1.05 1.55) (end 8.55 1.55) (layer "F.CrtYd") (width 0.05))
-    (fp_line (start -1.05 -1.55) (end -1.05 1.55) (layer "F.CrtYd") (width 0.05))
-    (fp_line (start 8.55 1.55) (end 8.55 -1.55) (layer "F.CrtYd") (width 0.05))
-    (fp_line (start 8.55 -1.55) (end -1.05 -1.55) (layer "F.CrtYd") (width 0.05))
-    (fp_line (start 0 0) (end 1.85 0) (layer "F.Fab") (width 0.1))
-    (fp_line (start 7.5 0) (end 5.65 0) (layer "F.Fab") (width 0.1))
-    (fp_line (start 5.65 -1.3) (end 1.85 -1.3) (layer "F.Fab") (width 0.1))
-    (fp_line (start 5.65 1.3) (end 5.65 -1.3) (layer "F.Fab") (width 0.1))
-    (fp_line (start 1.85 1.3) (end 5.65 1.3) (layer "F.Fab") (width 0.1))
-    (fp_line (start 1.85 -1.3) (end 1.85 1.3) (layer "F.Fab") (width 0.1))
-    (pad "1" thru_hole circle (at 0 0) (size 1.6 1.6) (drill 0.8) (layers *.Cu *.Mask)
+    (fp_text reference "C1" (at 4.258 2.54) (layer "F.SilkS")
+      (effects (font (size 1 1) (thickness 0.15)))
+    )
+    (fp_text value "10uF" (at 0.75 3.25) (layer "F.Fab")
+      (effects (font (size 1 1) (thickness 0.15)))
+    )
+    (fp_text user "${REFERENCE}" (at 0.75 0) (layer "F.Fab")
+      (effects (font (size 0.8 0.8) (thickness 0.12)))
+    )
+    (fp_circle (center 0.75 0) (end 2.87 0) (layer "F.SilkS") (width 0.12) (fill none))
+    (fp_circle (center 0.75 0) (end 3 0) (layer "F.CrtYd") (width 0.05) (fill none))
+    (fp_circle (center 0.75 0) (end 2.75 0) (layer "F.Fab") (width 0.1) (fill none))
+    (pad "1" thru_hole circle (at 0 0) (size 1.2 1.2) (drill 0.6) (layers *.Cu *.Mask)
       (net 2 "PWR3x3") (pintype "passive"))
-    (pad "2" thru_hole oval (at 7.5 0) (size 1.6 1.6) (drill 0.8) (layers *.Cu *.Mask)
+    (pad "2" thru_hole circle (at 1.5 0) (size 1.2 1.2) (drill 0.6) (layers *.Cu *.Mask)
       (net 1 "GND") (pintype "passive"))
-    (model "${KICAD6_3DMODEL_DIR}/Capacitor_THT.3dshapes/C_Axial_L3.8mm_D2.6mm_P7.50mm_Horizontal.wrl"
+    (model "${KICAD6_3DMODEL_DIR}/Capacitor_THT.3dshapes/C_Radial_D4.0mm_H5.0mm_P1.50mm.wrl"
       (offset (xyz 0 0 0))
       (scale (xyz 1 1 1))
@@
     (effects (font (size 1.5 1.5) (thickness 0.3)))
   )
-  (gr_text "github.com/SteffMUC/openDTUwDisplay \n[2023-01-27]" (at 161.036 94.996 90) (layer "B.Cu")
+  (gr_text "github.com/SteffMUC/openDTU_wDisplay\n[2023-01-27]" (at 161.036 94.996 90) (layer "B.Cu")
     (effects (font (size 1.5 1.5) (thickness 0.3)) (justify mirror))
   )
